File: ESP32-S3 Small Camera.kicad_sch (KiCad schematic)
At the start: 93 parts, among them J1 Conn_01x24, J2 U.FL Antenna Conn, J3 Conn_01x08, J4 Test Pad RST BOOT, Q1 FS8205A, U1 TLV73328PDQNR, U10 TLV73328PDQNR, U11 SN74LVC1T45DCK, U12 SN74LVC1T45DCK, U13 SN74LVC1T45DCK, U2 USBLC6-2SC6, U3 BQ25180YBGR, U4 TPS62840YBGR, U5 BQ27441-G1, U6 DW01A, U7 W25Q128JVP, U8 ESP32-S3R8, U9 TLV73315PDQNR, X1 40MHz, 15pF

Commit message: Rerouted, cleaned up
Parts:
- removed C35, C38: 100nF, Capacitor_SMD:C_0201_0603Metric, symbol Device:C_Small
Connections:
- net D+X: now also J3.5 (Pin_5); no longer J3.4 (Pin_4)
- net D-X: now also J3.4 (Pin_4); no longer J3.5 (Pin_5)

Commit message: Manufacturing Files Updated
Parts:
- C14, C39: footprint Capacitor_SMD:C_0402_1005Metric -> PCM_JLCPCB:C_0402
- L5: LCSC C317665 -> C3032791
Changed lines of the file:
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@@
 			)
 		)
-		(property "Footprint" "Capacitor_SMD:C_0402_1005Metric"
+		(property "Footprint" "PCM_JLCPCB:C_0402"
 			(at 141.732 34.29 90)
 			(hide yes)
@@
 			)
 		)
-		(property "Footprint" "Capacitor_SMD:C_0402_1005Metric"
+		(property "Footprint" "PCM_JLCPCB:C_0402"
 			(at 117.602 34.29 90)
 			(hide yes)
@@
 			)
 		)
-		(property "Description" "1.04A 18@250MHz 2nH 6GHz 70mΩ ±10% 0402 Inductors (SMD) ROHS"
+		(property "Description" "2nH 6GHz 8@100MHz 900mA 90mΩ Multilayer inductor、High-frequency inductor 0402 Inductors (SMD) ROHS"
 			(at 127 39.37 0)
 			(hide yes)
@@
 			)
 		)
-		(property "LCSC" "C317665"
+		(property "LCSC" "C3032791"
 			(at 127 39.37 90)
 			(hide yes)
